Commit message: Cập nhật dự án, dọn dẹp core dump

File: src/mir_robot/mir_description/urdf/include/mir_v1.urdf.xacro (robot description, xacro)
@@ -8,4 +8,5 @@
   <xacro:include filename="$(find mir_description)/urdf/include/mir.transmission.xacro" />
   <xacro:include filename="$(find mir_description)/urdf/include/sick_s300.urdf.xacro" />
+  <xacro:include filename="$(find mir_description)/urdf/include/realsense.urdf.xacro" />
   <xacro:property name="deg_to_rad" value="0.017453293" />
   <!-- The inertia for the MiR platform is intentionally chosen to be smaller than
@@ -266,4 +267,9 @@
     <!-- set the gazebo friction parameters for the wheels -->
     <xacro:set_all_wheel_frictions prefix="${prefix}"/>
+      <!-- Camera Realsense -->
+    <xacro:realsense_camera prefix="${prefix}" parent="${prefix}surface">
+      <!-- origin xyz="0.4 0 0.1" rpy="0 0 0" / -->
+      <origin xyz="0.30 0.0 0.15" rpy="0 0 0" />
+    </xacro:realsense_camera>
     <xacro:p3d_base_controller prefix="${prefix}" />
   </xacro:macro>
